Commit message: added gazebo to the Dockerfile and added the bringup package Added valid inertia to the A_00036.urdf, so that gazebo can work with it
Signed-off-by: Fabian Finkbeiner <fabian.finkbeiner@hs-heilbronn.de>

File: src/descriptions/urdf/A_00036-02.urdf (robot description, URDF)
Before this commit: robot DELTA_4DoF_γ, 27 links, 26 joints
Links:
- link tool0: mass 0 -> 0.001
- link tool_holder: geometry visual mesh filename=package://descriptions/meshes/A_00036/Unterarmverbinder.stl scale=0.001 0.001 0.001; visual mesh filename=package://descriptions/meshes/A_00036/Unterarmverbinder.stl scale=0.001 0.001 0.001
